File: t3-harness-adapter/t3-harness-adapter.kicad_pcb (KiCad board)
At the start: 2 copper layers, 61.9 x 49 mm, 13 parts, among them J1 Conn_01x14_Pin, J10 Conn_01x14_Pin, J11 Conn_01x14_Pin, J12 Conn_01x14_Pin, J13 Conn_01x14_Pin, J2 Conn_01x14_Pin, J3 Conn_01x14_Pin, J4 Conn_01x08_Pin, J5 Conn_01x08_Pin, J6 Conn_01x14_Pin, J7 Conn_01x14_Pin, J8 Conn_01x14_Pin, J9 Conn_01x14_Pin

Commit message: [pcb] added layout
Parts:
- moved J4 7.98 mm to (89.6, 86.6), turned to 0 degrees
- moved J5 7.82 mm to (144.3, 94.2), turned to 180 degrees
Routing:
- net /temperature: track 0.00 -> 82.5 mm
- net /fuel: track 0.00 -> 81.5 mm
- net /conn_1: track 0.00 -> 81.3 mm, vias 0 -> 2
- net /free_temp: track 0.00 -> 75.4 mm
- net /plus_clock: track 0.00 -> 74.9 mm, vias 0 -> 1
- net /charge: track 0.00 -> 74.3 mm
- net /indicator: track 0.00 -> 72.6 mm, vias 0 -> 1
- net /pressure_low: track 0.00 -> 68.1 mm
- net /pressure_hi: track 0.00 -> 66.9 mm, vias 0 -> 1
- net /high_beam: track 0.00 -> 66.7 mm, vias 0 -> 1
- net /instrument_light: track 0.00 -> 64.4 mm
- net /aux: track 0.00 -> 63.3 mm, vias 0 -> 1
- net /plus: track 0.00 -> 13.1 mm, vias 0 -> 2
- net /minus: vias 0 -> 3
- added copper zone on B.Cu, net /minus
- added copper zone on F.Cu, net /plus
