File: hw/disco-tft-adapter/disco_tft_adapter.kicad_pcb (KiCad board)
At the start: 4 copper layers, 127 x 116.1 mm, 34 parts, among them J1 QTH-030-02-L-D-A, J2 F31L-1A7H1-11030

Commit message: [layout] update revision to "Rev. B", rearrange silkscreen and some traces in order to pass DRC without flaws
Other:
- board text added: "Disco TFT Adapter Rev. B"
- board text removed: "Disco TFT Adapter Rev. A"
